File: 6segment.kicad_pcb (KiCad board)
At the start: 2 copper layers, 99.1 x 99.1 mm, 53 parts, among them J1 LA, J2 RA, J3 LK, J4 RK, J5 SS, J6 DS1, Q1 A, Q2 B, Q21 D1, Q22 D1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

Commit message: Update to KiCad v8
Connections:
- D11 pad 3: Net-(D11-Pad3) -> unconnected-(D11-Pad3)
- D11 pad 4: Net-(D11-Pad4) -> unconnected-(D11-Pad4)
- D11 pad 5: Net-(D11-Pad5) -> unconnected-(D11-Pad5)
- D111 pad 3: Net-(D111-Pad3) -> unconnected-(D111-Pad3)
- D111 pad 4: Net-(D111-Pad4) -> unconnected-(D111-Pad4)
- D111 pad 5: Net-(D111-Pad5) -> unconnected-(D111-Pad5)
- D112 pad 3: Net-(D112-Pad3) -> unconnected-(D112-Pad3)
- D112 pad 4: Net-(D112-Pad4) -> unconnected-(D112-Pad4)
- D112 pad 5: Net-(D112-Pad5) -> unconnected-(D112-Pad5)
- D113 pad 3: Net-(D113-Pad3) -> unconnected-(D113-Pad3)
- D113 pad 4: Net-(D113-Pad4) -> unconnected-(D113-Pad4)
- D113 pad 5: Net-(D113-Pad5) -> unconnected-(D113-Pad5)
- D114 pad 3: Net-(D114-Pad3) -> unconnected-(D114-Pad3)
- D114 pad 4: Net-(D114-Pad4) -> unconnected-(D114-Pad4)
- D114 pad 5: Net-(D114-Pad5) -> unconnected-(D114-Pad5)
- D115 pad 3: Net-(D115-Pad3) -> unconnected-(D115-Pad3)
- D115 pad 4: Net-(D115-Pad4) -> unconnected-(D115-Pad4)
- D115 pad 5: Net-(D115-Pad5) -> unconnected-(D115-Pad5)
- D116 pad 3: Net-(D116-Pad3) -> unconnected-(D116-Pad3)
- D116 pad 4: Net-(D116-Pad4) -> unconnected-(D116-Pad4)
- D116 pad 5: Net-(D116-Pad5) -> unconnected-(D116-Pad5)
- D117 pad 3: Net-(D117-Pad3) -> unconnected-(D117-Pad3)
- D117 pad 4: Net-(D117-Pad4) -> unconnected-(D117-Pad4)
- D117 pad 5: Net-(D117-Pad5) -> unconnected-(D117-Pad5)
- D12 pad 3: Net-(D12-Pad3) -> unconnected-(D12-Pad3)
- D12 pad 4: Net-(D12-Pad4) -> unconnected-(D12-Pad4)
- D12 pad 5: Net-(D12-Pad5) -> unconnected-(D12-Pad5)
- D13 pad 3: Net-(D13-Pad3) -> unconnected-(D13-Pad3)
- D13 pad 4: Net-(D13-Pad4) -> unconnected-(D13-Pad4)
- D13 pad 5: Net-(D13-Pad5) -> unconnected-(D13-Pad5)
- D14 pad 3: Net-(D14-Pad3) -> unconnected-(D14-Pad3)
- D14 pad 4: Net-(D14-Pad4) -> unconnected-(D14-Pad4)
- D14 pad 5: Net-(D14-Pad5) -> unconnected-(D14-Pad5)
- D15 pad 3: Net-(D15-Pad3) -> unconnected-(D15-Pad3)
- D15 pad 4: Net-(D15-Pad4) -> unconnected-(D15-Pad4)
- D15 pad 5: Net-(D15-Pad5) -> unconnected-(D15-Pad5)
- D16 pad 3: Net-(D16-Pad3) -> unconnected-(D16-Pad3)
- D16 pad 4: Net-(D16-Pad4) -> unconnected-(D16-Pad4)
- D16 pad 5: Net-(D16-Pad5) -> unconnected-(D16-Pad5)
- R21 pad 2: Net-(R21-Pad2) -> unconnected-(R21-Pad2)
- R22 pad 2: Net-(R22-Pad2) -> unconnected-(R22-Pad2)
Routing:
- net unconnected-(D116-Pad5): track 0.00 -> 12.3 mm
- net unconnected-(D113-Pad5): track 0.00 -> 12.3 mm
- net Net-(D116-Pad5): track 12.3 -> 0.00 mm
- net Net-(D113-Pad5): track 12.3 -> 0.00 mm
- net unconnected-(D16-Pad5): track 0.00 -> 12.3 mm
- net unconnected-(D13-Pad5): track 0.00 -> 12.3 mm
- net Net-(D16-Pad5): track 12.3 -> 0.00 mm
- net Net-(D13-Pad5): track 12.3 -> 0.00 mm
- net unconnected-(D117-Pad4): track 0.00 -> 10.3 mm
- net Net-(D117-Pad4): track 10.3 -> 0.00 mm
- net unconnected-(D12-Pad5): track 0.00 -> 6.56 mm
- net Net-(D12-Pad5): track 6.56 -> 0.00 mm
- net unconnected-(D15-Pad5): track 0.00 -> 6.56 mm
- net Net-(D15-Pad5): track 6.56 -> 0.00 mm
- net unconnected-(D15-Pad3): track 0.00 -> 6.56 mm
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Other:
- net class Default removed
- net class POWER removed
